File: BigBoyBoard/BBB_eagle.sch (EAGLE design)
At the start: 4 parts

Commit message: Design review 12/1
Parts:
- added C10, C11: 4.7uF, SparkFun-Capacitors:4.7UF0603
- added C12, C13, C16, C7: 100nF, SparkFun-Capacitors:4.7UF0603
- added C14: 0.01uf, SparkFun-Capacitors:4.7UF0603
- added C15, C99: 1uF, SparkFun-Capacitors:4.7UF0603
- added C17, C18: 18pF, SparkFun-Capacitors:4.7UF0603
- added C5: 4.7nF, SparkFun-Capacitors:0.1UF-0603-25V-(+80/-20%)
- added LED1: (no value), led:LEDCHIP-LED0805
- added R0: 0Ω, rcl:R-US_R0603
- added R1: 1KΩ, rcl:R-US_R0603
- added R10, R11: 60, SparkFun-Resistors:1KOHM-0603-1/10W-1%
- added R4, R6: 0, SparkFun-Resistors:1KOHM-0603-1/10W-1%
- added R5: 47k, SparkFun-Resistors:1KOHM-0603-1/10W-1%
- added RESET1: SWITCH, DiscreteComponents:SWITCH
- added RSH1, RSH2, RSH3, RSH7: 1 mΩ, INA4181A4:CSS2H-2512
- added SV2: (no value), con-lsta:FE05-1
- added U$14: INA4181A4, INA4181A4:INA4181A4
- added U$5: STM32F042K6T6, PI_Shield_Library:STM32F042K6T6
- added U$6: ET60T_2, ET60T:ET60T_2
- added U$7: AFRO_20A_ESC, afro_20A_esc:AFRO_20A_ESC
- added U$8: TCAN337D, PI_Shield_Library:TCAN337D
- added Y2: ECS-80-S-4X, ECS-80-S-4X:ECS-80-S-4X
- U$4: value STM32F042K6T6 -> ET60T_1; device PI_Shield_Library:STM32F042K6T6 -> ET60T:ET60T_1
Connections:
- new net +12V: RSH1.2, RSH2.2, RSH3.2, RSH7.2, U$14.IN+1, U$14.IN+2, U$14.IN+3, U$14.IN+4, U$4G$1.B15, U$4G$1.B16, U$4G$1.B7, U$4G$1.B8, U$6G$2.S1
- new net +3V3: C10.1, C11.1, C12.1, C13.1, C14.1, C15.1, C7.1, C99.1, R5.2, SV2.5, U$14.VS, U$5.VDD, U$5.VDDA, U$5.VDDIO2, U$6G$2.S5, U$8.VCC
- new net +5V: U$4G$1.B11, U$4G$1.B12, U$4G$1.B19, U$4G$1.B20, U$6G$2.S3
- new net +5VGND: U$4G$1.B10, U$4G$1.B17, U$4G$1.B18, U$4G$1.B9, U$6G$2.S4
- new net ADC_IN0: U$14.OUT4, U$5.PA0
- new net ADC_IN1: U$14.OUT3, U$5.PA1
- new net ADC_IN2: U$14.OUT1, U$5.PA2
- new net ADC_IN3: U$14.OUT2, U$5.PA3
- new net CAN_H: R10.2, U$4G$1.B24, U$8.CANH
- new net CAN_L: R11.1, U$4G$1.B23, U$8.CANL
- new net CAN_RX: U$5.PA11, U$8.TXD
- new net CAN_TX: U$5.PA12, U$8.RXD
- new net ESC1_R1: U$1.RED, U$4G$3.S1
- new net ESC1_R2: U$1.YEL, U$4G$3.S2
- new net ESC1_R3: U$1.BLK, U$4G$3.S3
- new net ESC2_L1: U$2.RED, U$4G$2.S1
- new net ESC2_L2: U$2.YEL, U$4G$2.S2
- new net ESC2_L3: U$2.BLK, U$4G$2.S3
- new net ESC3_R4: U$3.RED, U$4G$3.S4
- new net ESC3_R5: U$3.YEL, U$4G$3.S5
- new net ESC3_R6: U$3.BLK, U$4G$3.S6
- new net ESC7_L4: U$4G$2.S4, U$7.RED
- new net ESC7_L5: U$4G$2.S5, U$7.YEL
- new net ESC7_L6: U$4G$2.S6, U$7.BLK
- new net GND: C5.1, C7.2, R0.2, U$1.GND, U$1.PWM_GND, U$2.GND, U$2.PWM_GND, U$3.GND, U$3.PWM_GND, U$4G$1.B13, U$4G$1.B14, U$4G$1.B21, U$4G$1.B22, U$6G$2.S2, U$7.GND, U$7.PWM_GND, U$8.GND
- new net GNDA: C10.2, C11.2, C12.2, C13.2, C14.2, C15.2, C16.2, C17.2, C18.2, C99.2, LED1.C, R0.1, RESET1.P$1, SV2.1, U$14.GND, U$14.REF1, U$14.REF2, U$14.REF3, U$14.REF4, U$5.PB8-BOOT0, U$5.VSS, U$5.VSS1, U$6G$2.S6
- new net N$1: R1.1, U$5.PA15
- new net N$12: U$4G$1.B6
- new net N$13: U$4G$1.B5
- new net N$14: U$4G$1.B4
- new net N$15: U$4G$1.B3
- new net N$16: U$4G$1.B2
- new net N$17: U$4G$1.B1
- new net N$2: LED1.A, R1.2
- new net N$3: C18.1, R4.1, Y2.2
- new net N$30: U$6G$1.B24
- new net N$31: U$6G$1.B23
- new net N$32: U$6G$1.B22
- new net N$33: U$6G$1.B21
- new net N$34: U$6G$1.B20
- new net N$35: U$6G$1.B19
- new net N$36: U$6G$1.B18
- new net N$37: U$6G$1.B17
- new net N$38: U$6G$1.B16
- new net N$39: U$6G$1.B15
- new net N$4: C17.1, R6.1, Y2.1
- new net N$40: U$6G$1.B14
- new net N$41: U$6G$1.B13
- new net N$42: U$6G$1.B1
- new net N$43: U$6G$1.B2
- new net N$44: U$6G$1.B3
- new net N$45: U$6G$1.B4
- new net N$46: U$6G$1.B5
- new net N$47: U$6G$1.B6
- new net N$48: U$6G$1.B7
- new net N$49: U$6G$1.B8
- new net N$5: C5.2, R10.1, R11.2
- new net N$50: U$6G$1.B9
- new net N$51: U$6G$1.B10
- new net N$52: U$6G$1.B11
- new net N$53: U$6G$1.B12
- new net N$58: U$14.NC.
- new net NRST: C16.1, R5.1, RESET1.P$2, SV2.2, U$5.NRST
- new net OSC_IN: R6.2, U$5.PF0-OSC_IN
- new net OSC_OUT: R4.2, U$5.PF1-OSC_OUT
- new net SWCLK: SV2.3, U$5.PA14
- new net SWDIO: SV2.4, U$5.PA13
- new net TIM3_CH1: U$5.PA6, U$7.PWM_SGN
- new net TIM3_CH2: U$2.PWM_SGN, U$5.PA7
- new net TIM3_CH3: U$1.PWM_SGN, U$5.PB0
- new net TIM3_CH4: U$3.PWM_SGN, U$5.PB1
- new net VCC1: RSH1.1, U$1.VCC, U$14.IN-2
- new net VCC2: RSH2.1, U$14.IN-4, U$2.VCC
- new net VCC3: RSH3.1, U$14.IN-1, U$3.VCC
- new net VCC7: RSH7.1, U$14.IN-3, U$7.VCC
Other:
- note added: "CAN TERMINATION"
- note added: "CAN TRANSCEIVER"
- note added: "Pin 1 (VDD)"
- note added: "Pin 17 (VDDIO2)"
- note added: "Pin 5 (VDDA)"
- moved on the sheet: U$1, U$2, U$3

Commit message: Tenatively compleated esc board
Connections:
- removed net N$30: U$6G$1.B24
- removed net N$31: U$6G$1.B23
- removed net N$32: U$6G$1.B22
- removed net N$33: U$6G$1.B21
- removed net N$34: U$6G$1.B20
- removed net N$35: U$6G$1.B19
- removed net N$36: U$6G$1.B18
- removed net N$37: U$6G$1.B17
- removed net N$38: U$6G$1.B16
- removed net N$39: U$6G$1.B15
- removed net N$40: U$6G$1.B14
- removed net N$41: U$6G$1.B13
- removed net N$42: U$6G$1.B1
- removed net N$43: U$6G$1.B2
- removed net N$44: U$6G$1.B3
- removed net N$45: U$6G$1.B4
- removed net N$46: U$6G$1.B5
- removed net N$47: U$6G$1.B6
- removed net N$48: U$6G$1.B7
- removed net N$49: U$6G$1.B8
- removed net N$50: U$6G$1.B9
- removed net N$51: U$6G$1.B10
- removed net N$52: U$6G$1.B11
- removed net N$53: U$6G$1.B12
- net +12V: now also U$6.S6; no longer U$6G$2.S1
- net +3V3: now also U$6.S5; no longer U$6G$2.S5
- net +5V: now also U$6.S3; no longer U$6G$2.S3
- net +5VGND: now also U$6.S4; no longer U$6G$2.S4
- net GND: now also U$6.S2; no longer U$6G$2.S2
- net GNDA: now also U$6.S1; no longer U$6G$2.S6
Other:
- moved on the sheet: C99

Commit message: 12/27 updates
Connections:
- removed net N$12: U$4G$1.B6
- removed net N$13: U$4G$1.B5
- removed net N$14: U$4G$1.B4
- removed net N$15: U$4G$1.B3
- removed net N$16: U$4G$1.B2
- removed net N$17: U$4G$1.B1
- net +5V: now also U$4G$1.B3, U$4G$1.B4
- net +5VGND: now also U$4G$1.B1, U$4G$1.B2
- net GND: now also U$4G$1.B5, U$4G$1.B6
Changed lines of the file:
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@@
 <pinref part="U$4" gate="G$1" pin="B21"/>
 <wire x1="43.18" y1="48.26" x2="50.8" y2="48.26" width="0.1524" layer="91"/>
-<label x="43.18" y="45.72" size="1.778" layer="95"/>
 </segment>
 <segment>
 <pinref part="U$4" gate="G$1" pin="B22"/>
 <wire x1="43.18" y1="53.34" x2="50.8" y2="53.34" width="0.1524" layer="91"/>
-<label x="45.72" y="50.8" size="1.778" layer="95"/>
 </segment>
 <segment>
@@
 <wire x1="43.18" y1="12.7" x2="50.8" y2="12.7" width="0.1524" layer="91"/>
 <label x="45.72" y="10.16" size="1.778" layer="95"/>
+</segment>
+<segment>
+<pinref part="U$4" gate="G$1" pin="B5"/>
+<wire x1="17.78" y1="27.94" x2="10.16" y2="27.94" width="0.1524" layer="91"/>
+<label x="10.16" y="25.4" size="1.778" layer="95"/>
+</segment>
+<segment>
+<pinref part="U$4" gate="G$1" pin="B6"/>
+<wire x1="17.78" y1="33.02" x2="10.16" y2="33.02" width="0.1524" layer="91"/>
+<label x="10.16" y="30.48" size="1.778" layer="95"/>
 </segment>
 </net>
@@
 <pinref part="U$4" gate="G$1" pin="B19"/>
 <wire x1="43.18" y1="38.1" x2="50.8" y2="38.1" width="0.1524" layer="91"/>
-<label x="45.72" y="35.56" size="1.778" layer="95"/>
 </segment>
 <segment>
 <pinref part="U$4" gate="G$1" pin="B20"/>
 <wire x1="43.18" y1="43.18" x2="50.8" y2="43.18" width="0.1524" layer="91"/>
-<label x="45.72" y="40.64" size="1.778" layer="95"/>
+</segment>
+<segment>
+<pinref part="U$4" gate="G$1" pin="B3"/>
+<wire x1="17.78" y1="17.78" x2="10.16" y2="17.78" width="0.1524" layer="91"/>
+<label x="10.16" y="15.24" size="1.778" layer="95"/>
+</segment>
+<segment>
+<pinref part="U$4" gate="G$1" pin="B4"/>
+<wire x1="17.78" y1="22.86" x2="10.16" y2="22.86" width="0.1524" layer="91"/>
+<label x="10.16" y="20.32" size="1.778" layer="95"/>
 </segment>
 </net>
@@
 <pinref part="U$4" gate="G$1" pin="B17"/>
 <wire x1="43.18" y1="27.94" x2="50.8" y2="27.94" width="0.1524" layer="91"/>
-<label x="43.18" y="25.4" size="1.778" layer="95"/>
 </segment>
 <segment>
 <pinref part="U$4" gate="G$1" pin="B18"/>
 <wire x1="43.18" y1="33.02" x2="50.8" y2="33.02" width="0.1524" layer="91"/>
-<label x="43.18" y="30.48" size="1.778" layer="95"/>
+</segment>
+<segment>
+<pinref part="U$4" gate="G$1" pin="B1"/>
+<wire x1="17.78" y1="7.62" x2="10.16" y2="7.62" width="0.1524" layer="91"/>
+<label x="10.16" y="5.08" size="1.778" layer="95"/>
+</segment>
+<segment>
+<pinref part="U$4" gate="G$1" pin="B2"/>
+<wire x1="17.78" y1="12.7" x2="10.16" y2="12.7" width="0.1524" layer="91"/>
+<label x="10.16" y="10.16" size="1.778" layer="95"/>
 </segment>
 </net>
@@
 </segment>
 </net>
-<net name="N$12" class="0">
-<segment>
-<pinref part="U$4" gate="G$1" pin="B6"/>
-<wire x1="17.78" y1="33.02" x2="10.16" y2="33.02" width="0.1524" layer="91"/>
-</segment>
-</net>
-<net name="N$13" class="0">
-<segment>
-<pinref part="U$4" gate="G$1" pin="B5"/>
-<wire x1="17.78" y1="27.94" x2="10.16" y2="27.94" width="0.1524" layer="91"/>
-</segment>
-</net>
-<net name="N$14" class="0">
-<segment>
-<pinref part="U$4" gate="G$1" pin="B4"/>
-<wire x1="17.78" y1="22.86" x2="10.16" y2="22.86" width="0.1524" layer="91"/>
-</segment>
-</net>
-<net name="N$15" class="0">
-<segment>
-<pinref part="U$4" gate="G$1" pin="B3"/>
-<wire x1="17.78" y1="17.78" x2="10.16" y2="17.78" width="0.1524" layer="91"/>
-</segment>
-</net>
-<net name="N$16" class="0">
-<segment>
-<pinref part="U$4" gate="G$1" pin="B2"/>
-<wire x1="17.78" y1="12.7" x2="10.16" y2="12.7" width="0.1524" layer="91"/>
-</segment>
-</net>
-<net name="N$17" class="0">
-<segment>
-<pinref part="U$4" gate="G$1" pin="B1"/>
-<wire x1="17.78" y1="7.62" x2="10.16" y2="7.62" width="0.1524" layer="91"/>
-</segment>
-</net>

Commit message: change
Connections:
- new net NC1: U$4G$1.B17
- new net NC2: U$4G$1.B18
- new net NC3: U$4G$1.B19
- new net NC4: U$4G$1.B20
- net +5V: no longer U$4G$1.B19, U$4G$1.B20
- net +5VGND: no longer U$4G$1.B17, U$4G$1.B18
Changed lines of the file:
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@@
-</segment>
-<segment>
-<pinref part="U$4" gate="G$1" pin="B19"/>
-<wire x1="43.18" y1="38.1" x2="50.8" y2="38.1" width="0.1524" layer="91"/>
-</segment>
-<segment>
-<pinref part="U$4" gate="G$1" pin="B20"/>
-<wire x1="43.18" y1="43.18" x2="50.8" y2="43.18" width="0.1524" layer="91"/>
 </segment>
 <segment>
@@
 <wire x1="17.78" y1="53.34" x2="10.16" y2="53.34" width="0.1524" layer="91"/>
 <label x="10.16" y="50.8" size="1.778" layer="95"/>
-</segment>
-<segment>
-<pinref part="U$4" gate="G$1" pin="B17"/>
-<wire x1="43.18" y1="27.94" x2="50.8" y2="27.94" width="0.1524" layer="91"/>
-</segment>
-<segment>
-<pinref part="U$4" gate="G$1" pin="B18"/>
-<wire x1="43.18" y1="33.02" x2="50.8" y2="33.02" width="0.1524" layer="91"/>
 </segment>
 <segment>
@@
 </segment>
 </net>
+<net name="NC1" class="0">
+<segment>
+<pinref part="U$4" gate="G$1" pin="B17"/>
+<wire x1="43.18" y1="27.94" x2="50.8" y2="27.94" width="0.1524" layer="91"/>
+<label x="45.72" y="25.4" size="1.778" layer="95"/>
+</segment>
+</net>
+<net name="NC2" class="0">
+<segment>
+<pinref part="U$4" gate="G$1" pin="B18"/>
+<wire x1="43.18" y1="33.02" x2="50.8" y2="33.02" width="0.1524" layer="91"/>
+<label x="45.72" y="30.48" size="1.778" layer="95"/>
+</segment>
+</net>
+<net name="NC3" class="0">
+<segment>
+<pinref part="U$4" gate="G$1" pin="B19"/>
+<wire x1="43.18" y1="38.1" x2="50.8" y2="38.1" width="0.1524" layer="91"/>
+<label x="45.72" y="35.56" size="1.778" layer="95"/>
+</segment>
+</net>
+<net name="NC4" class="0">
+<segment>
+<pinref part="U$4" gate="G$1" pin="B20"/>
+<wire x1="43.18" y1="43.18" x2="50.8" y2="43.18" width="0.1524" layer="91"/>
+<label x="48.26" y="40.64" size="1.778" layer="95"/>
+</segment>
+</net>
