File: BigBoyBoard/BBB_eagle.brd (EAGLE design)
At the start: 94 x 87.1 mm, 36 parts, among them Y2 ECS-80-S-4X

Commit message: 12/27 updates
Parts:
- moved R11 4.00 mm to (4.89, 72.4)
- moved R10 4.00 mm to (9.08, 72.4)
- moved C15 0.17 mm to (29.2, 60.7)
- moved C11 0.15 mm to (32.8, 60.7)
Connections:
- removed net N$12: U$4.B6
- removed net N$13: U$4.B5
- removed net N$14: U$4.B4
- removed net N$15: U$4.B3
- removed net N$16: U$4.B2
- removed net N$17: U$4.B1
- net +5V: now also U$4.B3, U$4.B4
- net +5VGND: now also U$4.B1, U$4.B2
- net GND: now also U$4.B5, U$4.B6
Routing:
- net CAN_H: track 96.1 -> 113.3 mm, vias 0 -> 1
- net GNDA: track 196.5 -> 187.3 mm, vias 7 -> 6
- net +12V: track 240.1 -> 248.4 mm
- net TIM3_CH3: track 84.6 -> 79.9 mm
- net VCC7: track 30.5 -> 33.5 mm
- net CAN_L: track 108.7 -> 110.9 mm
- net ADC_IN2: track 11.3 -> 13.3 mm
- net N$5: track 9.90 -> 8.61 mm
- net +5VGND: track 169.3 -> 168.1 mm
- net NRST: track 46.1 -> 47.3 mm
- net +3V3: track 204.3 -> 203.2 mm
- net +5V: track 171.5 -> 170.6 mm
- net GND: vias 7 -> 9

Commit message: change
Connections:
- new net NC1: U$4.B17
- new net NC2: U$4.B18
- new net NC3: U$4.B19
- new net NC4: U$4.B20
- net +5V: no longer U$4.B19, U$4.B20
- net +5VGND: no longer U$4.B17, U$4.B18
Changed lines of the file:
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@@
 <setting verticaltext="up"/>
 </settings>
-<grid distance="0.5" unitdist="mm" unit="mm" style="lines" multiple="1" display="no" altdistance="5" altunitdist="mil" altunit="mil"/>
+<grid distance="19.6850394" unitdist="mil" unit="mil" style="lines" multiple="1" display="no" altdistance="5" altunitdist="mil" altunit="mil"/>
 <layers>
 <layer number="1" name="Top" color="4" fill="1" visible="yes" active="yes"/>
@@
 <via x="21" y="80.5" extent="1-16" drill="0.8" diameter="1.15"/>
 <via x="22" y="77.5" extent="1-16" drill="0.8" diameter="1.15"/>
-<wire x1="21" y1="80.5" x2="22" y2="77.5" width="0" layer="19" extent="1-1"/>
 </signal>
 <signal name="NRST">
@@
 <wire x1="26.95" y1="46" x2="29" y2="46" width="0.4064" layer="1"/>
 <wire x1="29" y1="46" x2="30" y2="47" width="0.4064" layer="1"/>
-<wire x1="30" y1="48.5" x2="28.416" y2="50.084" width="0.4064" layer="1"/>
-<wire x1="28.416" y1="50.084" x2="28.416" y2="50.253" width="0.4064" layer="1"/>
-<wire x1="30" y1="47" x2="30" y2="48.5" width="0.4064" layer="1"/>
+<wire x1="30" y1="49" x2="28.747" y2="50.253" width="0.4064" layer="1"/>
+<wire x1="30" y1="47" x2="30" y2="49" width="0.4064" layer="1"/>
 <wire x1="26.67" y1="72.39" x2="26.67" y2="74.33" width="0.5" layer="1"/>
 <wire x1="26.67" y1="74.33" x2="26" y2="75" width="0.5" layer="1"/>
@@
 <via x="26.797" y="50.8" extent="1-16" drill="0.35"/>
 <wire x1="26.797" y1="50.8" x2="25.3174" y2="50.8" width="0.4064" layer="16"/>
+<wire x1="28.747" y1="50.253" x2="28.416" y2="50.253" width="0.4064" layer="1"/>
 </signal>
 <signal name="N$4">
@@
 <wire x1="42.293" y1="37.6" x2="62.61" y2="37.6" width="0.4064" layer="1"/>
 <wire x1="62.61" y1="37.6" x2="71" y2="29.21" width="0.4064" layer="1"/>
-<wire x1="23.1917" y1="51.775" x2="28.7002625" y2="51.775" width="0.508" layer="16"/>
+<wire x1="23.1917" y1="51.775" x2="28.7002625" y2="51.775" width="0.4064" layer="16"/>
 <wire x1="28.7002625" y1="51.775" x2="35.6616625" y2="44.8136" width="0.508" layer="16"/>
 <wire x1="35.6616625" y1="44.8136" x2="39.0064" y2="44.8136" width="0.508" layer="16"/>
@@
 <wire x1="38.6964" y1="56.1964" x2="39.5" y2="57" width="0.5" layer="16"/>
 <via x="20.57298125" y="48.4348" extent="1-16" drill="0.35"/>
-<wire x1="20.57298125" y1="48.4448" x2="18.55613125" y2="50.46165" width="0.5" layer="16"/>
+<wire x1="20.57298125" y1="48.4448" x2="18.55613125" y2="50.46165" width="0.4064" layer="16"/>
 <wire x1="20.57298125" y1="48.4348" x2="19.489" y2="49.51878125" width="0.5" layer="1"/>
 <wire x1="19.489" y1="49.51878125" x2="19.489" y2="51.878" width="0.5" layer="1"/>
 <via x="19.489" y="51.878" extent="1-16" drill="0.35"/>
 <wire x1="19.489" y1="51.878" x2="19.3692" y2="51.7582" width="0.5" layer="16"/>
-<wire x1="19.3692" y1="51.7582" x2="17.4315" y2="51.7582" width="0.5" layer="16"/>
+<wire x1="19.3692" y1="51.7582" x2="17.4315" y2="51.7582" width="0.4064" layer="16"/>
 <wire x1="20.57298125" y1="48.4348" x2="20.57298125" y2="48.4448" width="0.5" layer="16"/>
-<wire x1="18.55613125" y1="50.46165" x2="17.46165" y2="50.46165" width="0.5" layer="16"/>
+<wire x1="18.55613125" y1="50.46165" x2="17.46165" y2="50.46165" width="0.4064" layer="16"/>
 <wire x1="41.947" y1="37.946" x2="42.293" y2="37.6" width="0.4064" layer="1"/>
 </signal>
@@
 <wire x1="21.725" y1="52.975" x2="21.725" y2="51.8642" width="0.254" layer="1"/>
 <via x="21.725" y="51.8642" extent="1-16" drill="0.35"/>
-<wire x1="22.9358" y1="53.075" x2="23.1917" y2="53.075" width="0.254" layer="16"/>
+<wire x1="22.9358" y1="53.075" x2="23.1917" y2="53.075" width="0.4064" layer="16"/>
 <wire x1="23.1917" y1="53.075" x2="23.1167" y2="53" width="0.2032" layer="16"/>
 <wire x1="23.1167" y1="53" x2="22" y2="53" width="0.2032" layer="16"/>
@@
 <contactref element="U$4" pad="L6-2"/>
 <contactref element="U$4" pad="L6-6"/>
-<polygon width="0.254" layer="1" isolate="0.508">
+<polygon width="1.27" layer="1" isolate="0.508">
 <vertex x="1.27" y="34.29"/>
 <vertex x="1.27" y="30.48"/>
@@
 <contactref element="U$4" pad="L5-3"/>
 <contactref element="U$4" pad="L5-7"/>
-<polygon width="0.254" layer="1">
+<polygon width="1.27" layer="1">
 <vertex x="1.27" y="27.94"/>
 <vertex x="1.27" y="22.86"/>
@@
 <contactref element="U$4" pad="L4-7"/>
 <contactref element="U$4" pad="L4-9"/>
-<polygon width="0.254" layer="1">
+<polygon width="1.27" layer="1">
 <vertex x="1.27" y="20.32"/>
 <vertex x="1.27" y="16.51"/>
@@
 <contactref element="U$4" pad="L2-10"/>
 <contactref element="U$4" pad="L2-1"/>
-<polygon width="0.1524" layer="16">
+<polygon width="1.27" layer="16">
 <vertex x="7.62" y="1.27"/>
 <vertex x="11.43" y="1.27"/>
@@
 <contactref element="U$4" pad="L1-9"/>
 <contactref element="U$4" pad="L1-10"/>
-<polygon width="0.1524" layer="16">
+<polygon width="1.27" layer="16">
 <vertex x="2.04" y="40.64"/>
 <vertex x="2.04" y="38.2"/>
@@
 <vertex x="10.414" y="17.653"/>
 <vertex x="10.414" y="37.846"/>
-<vertex x="6.35" y="41.91"/>
-<vertex x="2.04" y="41.91"/>
+<vertex x="5.85" y="42.41"/>
+<vertex x="2.04" y="42.41"/>
 </polygon>
 </signal>
@@
 <contactref element="U$4" pad="B11"/>
 <contactref element="U$4" pad="B12"/>
-<contactref element="U$4" pad="B19"/>
-<contactref element="U$4" pad="B20"/>
 <wire x1="43.22" y1="6.74" x2="44.45" y2="6.74" width="0.508" layer="1"/>
 <wire x1="44.95" y1="6.74" x2="45.76" y2="6.74" width="0.508" layer="1"/>
@@
 <wire x1="45.3676125" y1="9.28" x2="45.76" y2="9.28" width="0.5" layer="1"/>
 <wire x1="17.9956125" y1="36.652" x2="45.3676125" y2="9.28" width="0.5" layer="1"/>
-<wire x1="43.22" y1="4.2" x2="45.76" y2="4.2" width="0" layer="19" extent="1-1"/>
-<wire x1="45.76" y1="6.74" x2="45.76" y2="4.2" width="0" layer="19" extent="1-1"/>
 </signal>
 <signal name="+5VGND">
 <contactref element="U$4" pad="B9"/>
 <contactref element="U$4" pad="B10"/>
-<contactref element="U$4" pad="B17"/>
-<contactref element="U$4" pad="B18"/>
 <wire x1="38.14" y1="6.74" x2="39.37" y2="6.74" width="0.508" layer="1"/>
 <wire x1="39.37" y1="6.74" x2="40.68" y2="6.74" width="0.508" layer="1"/>
@@
 <wire x1="39.285" y1="12.285" x2="40.68" y2="10.89" width="0.5" layer="1"/>
 <wire x1="40.68" y1="10.89" x2="40.68" y2="9.28" width="0.5" layer="1"/>
-<wire x1="38.14" y1="4.2" x2="40.68" y2="4.2" width="0" layer="19" extent="1-1"/>
-<wire x1="40.68" y1="6.74" x2="40.68" y2="4.2" width="0" layer="19" extent="1-1"/>
 </signal>
 <signal name="GNDA">
@@
 <via x="20.32" y="54.61" extent="1-16" drill="0.635"/>
 <wire x1="20.32" y1="54.61" x2="21.2452" y2="53.6848" width="0.508" layer="16"/>
-<wire x1="22.86" y1="53.6848" x2="21.5" y2="53.6848" width="0.508" layer="16"/>
+<wire x1="22.86" y1="53.6848" x2="21.5" y2="53.6848" width="0.4064" layer="16"/>
 <wire x1="21.5" y1="53.6848" x2="21.2452" y2="53.6848" width="0.508" layer="16"/>
-<wire x1="23.1917" y1="48.525" x2="23.1515" y2="48.5652" width="0.508" layer="16"/>
-<wire x1="23.1515" y1="48.5652" x2="22.0954125" y2="48.5652" width="0.508" layer="16"/>
-<wire x1="22.0954125" y1="48.5652" x2="20.32" y2="50.3406125" width="0.508" layer="16"/>
+<wire x1="20.32" y1="50.3406125" x2="22.0954125" y2="48.5652" width="0.508" layer="16"/>
 <wire x1="20.32" y1="50.3406125" x2="20.32" y2="51" width="0.508" layer="16"/>
 <wire x1="20.32" y1="51" x2="20.32" y2="54.61" width="0.508" layer="16"/>
@@
 <via x="25.4" y="46.99" extent="1-16" drill="0.35"/>
 <wire x1="25.4" y1="46.99" x2="25.4" y2="47.6866375" width="0.381" layer="16"/>
-<wire x1="24.5616375" y1="48.525" x2="23.1917" y2="48.525" width="0.381" layer="16"/>
+<wire x1="24.5616375" y1="48.525" x2="23.1917" y2="48.525" width="0.4064" layer="16"/>
 <wire x1="25.4" y1="47.6866375" x2="24.5616375" y2="48.525" width="0.381" layer="16"/>
 <wire x1="38.1" y1="69.469" x2="37.758" y2="69.469" width="0.508" layer="16"/>
@@
 <wire x1="32.778" y1="61.508" x2="32.676" y2="61.508" width="0.5" layer="16"/>
 <wire x1="20.32" y1="50.3406125" x2="19.8903875" y2="50.3406125" width="0.5" layer="16"/>
-<wire x1="19.1462" y1="51.0848" x2="17.4081" y2="51.0848" width="0.5" layer="16"/>
+<wire x1="19.1462" y1="51.0848" x2="17.4081" y2="51.0848" width="0.4064" layer="16"/>
 <wire x1="19.8903875" y1="50.3406125" x2="19.1462" y2="51.0848" width="0.5" layer="16"/>
 <wire x1="19.8948" y1="54.1848" x2="18.1848" y2="54.1848" width="0.5" layer="16"/>
-<wire x1="17.725" y1="53.725" x2="17.4483" y2="53.725" width="0.5" layer="16"/>
-<wire x1="18.1848" y1="54.1848" x2="17.725" y2="53.725" width="0.5" layer="16"/>
+<wire x1="17.725" y1="53.725" x2="17.4483" y2="53.725" width="0.4064" layer="16"/>
+<wire x1="18.1848" y1="54.1848" x2="17.725" y2="53.725" width="0.4064" layer="16"/>
+<wire x1="22.0954125" y1="48.5652" x2="22.1356125" y2="48.525" width="0.4064" layer="16"/>
+<wire x1="22.1356125" y1="48.525" x2="23.1917" y2="48.525" width="0.4064" layer="16"/>
 </signal>
 <signal name="CAN_H">
@@
 <via x="73" y="71.5" extent="1-16" drill="0.8" diameter="1.15"/>
 </signal>
+<signal name="NC1">
+<contactref element="U$4" pad="B17"/>
+</signal>
+<signal name="NC2">
+<contactref element="U$4" pad="B18"/>
+</signal>
+<signal name="NC3">
+<contactref element="U$4" pad="B19"/>
+</signal>
+<signal name="NC4">
+<contactref element="U$4" pad="B20"/>
+</signal>
 </signals>

Commit message: 12/30 update
Parts:
- moved C7 1.10 mm to (9.07, 78.8)
Routing:
- net +12V: track 248.4 -> 244.4 mm
- net VCC7: track 33.5 -> 30.6 mm
- net GNDA: track 187.3 -> 185.7 mm
- net GND: track 137.2 -> 136.6 mm, vias 9 -> 25
- net +3V3: track 203.4 -> 203.9 mm

Commit message: Update BigBoyBoard/BBB_eagle.brd
Routing:
- net TIM3_CH4: track 74.9 -> 82.0 mm, vias 1 -> 2
- net VCC3: track 72.6 -> 74.1 mm
- net GND: vias 25 -> 28
Changed lines of the file:
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@@
 <setting verticaltext="up"/>
 </settings>
-<grid distance="0.5" unitdist="mm" unit="mm" style="lines" multiple="1" display="no" altdistance="5" altunitdist="mil" altunit="mil"/>
+<grid distance="1" unitdist="mm" unit="mm" style="lines" multiple="1" display="no" altdistance="5" altunitdist="mil" altunit="mil"/>
 <layers>
 <layer number="1" name="Top" color="4" fill="1" visible="yes" active="yes"/>
@@
 <via x="2.5" y="85" extent="1-16" drill="0.35"/>
 <via x="11.5" y="82" extent="1-16" drill="0.35"/>
+<via x="80" y="45" extent="1-16" drill="0.35"/>
+<via x="80" y="40" extent="1-16" drill="0.35"/>
+<via x="86" y="37" extent="1-16" drill="0.35"/>
 </signal>
 <signal name="NRST">
@@
 <contactref element="U$5" pad="PB1"/>
 <contactref element="U$3" pad="PWM_SGN"/>
-<wire x1="91.12" y1="47.53" x2="78.96" y2="59.69" width="0.254" layer="16"/>
-<wire x1="78.96" y1="59.69" x2="50.8" y2="59.69" width="0.254" layer="16"/>
 <via x="49.022" y="51.308" extent="1-16" drill="0.35"/>
 <wire x1="49.022" y1="51.308" x2="48.006" y2="50.292" width="0.254" layer="1"/>
 <wire x1="48.006" y1="50.292" x2="39.878" y2="50.292" width="0.254" layer="1"/>
-<wire x1="50.8" y1="59.69" x2="49.022" y2="57.912" width="0.254" layer="16"/>
+<wire x1="49.022" y1="57.912" x2="50.8" y2="59.69" width="0.254" layer="16"/>
 <wire x1="49.022" y1="57.912" x2="49.022" y2="51.308" width="0.254" layer="16"/>
 <wire x1="32.92" y1="57.25" x2="32.92" y2="58.24" width="0.254" layer="1"/>
 <wire x1="39.878" y1="50.292" x2="32.92" y2="57.25" width="0.254" layer="1"/>
+<wire x1="50.8" y1="59.69" x2="75" y2="60" width="0.254" layer="16"/>
+<via x="75" y="60" extent="1-16" drill="0.35"/>
+<wire x1="75" y1="48" x2="75" y2="60" width="0.254" layer="1"/>
+<wire x1="91.12" y1="47.53" x2="75.47" y2="47.53" width="0.254" layer="1"/>
+<wire x1="75.47" y1="47.53" x2="75" y2="48" width="0.254" layer="1"/>
 </signal>
 <signal name="TIM3_CH3">
@@
 <via x="50.165" y="56.896" extent="1-16" drill="0.635"/>
 <wire x1="50.165" y1="56.896" x2="51.689" y2="58.42" width="0.254" layer="16"/>
-<wire x1="51.689" y1="58.42" x2="74.93" y2="58.42" width="0.254" layer="16"/>
-<via x="74.93" y="58.42" extent="1-16" drill="0.635"/>
-<wire x1="74.93" y1="58.42" x2="77.47" y2="55.88" width="0.254" layer="1"/>
-<wire x1="77.47" y1="55.88" x2="77.47" y2="52.07" width="0.254" layer="1"/>
+<wire x1="51.689" y1="58.42" x2="77.43" y2="58.42" width="0.254" layer="16"/>
+<via x="77.43" y="58.42" extent="1-16" drill="0.635"/>
+<wire x1="77.43" y1="58.42" x2="77.47" y2="58.38" width="0.254" layer="1"/>
+<wire x1="77.47" y1="58.38" x2="77.47" y2="52.07" width="0.254" layer="1"/>
 </signal>
 <signal name="VCC2">
@@
 <contactref element="U$4" pad="B20"/>
 </signal>
-<signal name="N$11">
-<via x="80" y="45" extent="1-16" drill="0.35"/>
-</signal>
-<signal name="N$12">
-<via x="80" y="40" extent="1-16" drill="0.35"/>
-</signal>
 </signals>

Commit message: Update BigBoyBoard/BBB_eagle.brd
Routing:
- net +5V: track 170.6 -> 169.1 mm
- net TIM3_CH1: track 36.9 -> 38.0 mm
- net CAN_H: track 113.3 -> 112.7 mm
- net GND: vias 28 -> 30
Changed lines of the file:
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@@
 <attribute name="VALUE" x="19.685" y="65.786" size="0.6096" layer="27" font="vector" ratio="20" rot="R270" align="top-center"/>
 </element>
-<element name="U$4" library="ET60T" package="ET60T_1" value="ET60T_1" x="47.03" y="6.74" smashed="yes"/>
+<element name="U$4" library="ET60T" package="ET60T_1" value="ET60T_1" x="46.99" y="6.74" smashed="yes"/>
 <element name="U$7" library="afro_20A_esc" package="AFRO_20A_ESC" value="AFRO_20A_ESC" x="21.59" y="25.4" smashed="yes">
 <attribute name="NAME" x="0.5" y="35.56" size="1.27" layer="25"/>
@@
 <contactref element="U$4" pad="B13"/>
 <contactref element="U$4" pad="B14"/>
-<wire x1="50.84" y1="6.74" x2="48.3" y2="6.74" width="0.8128" layer="1"/>
+<wire x1="50.8" y1="6.74" x2="48.26" y2="6.74" width="0.8128" layer="1"/>
 <wire x1="4.23" y1="76.2" x2="2.3876" y2="74.3576" width="0.508" layer="1"/>
 <wire x1="2.3876" y1="74.3576" x2="2.3876" y2="65.405" width="0.508" layer="1"/>
@@
 <contactref element="U$4" pad="B5"/>
 <contactref element="U$4" pad="B6"/>
-<wire x1="48.3" y1="9.28" x2="48.3" y2="6.74" width="0.8128" layer="1"/>
-<wire x1="48.3" y1="9.28" x2="50.84" y2="9.28" width="0.8128" layer="1"/>
-<wire x1="50.84" y1="9.28" x2="50.84" y2="6.74" width="0.8128" layer="1"/>
+<wire x1="48.26" y1="9.28" x2="48.26" y2="6.74" width="0.8128" layer="1"/>
+<wire x1="48.26" y1="9.28" x2="50.8" y2="9.28" width="0.8128" layer="1"/>
+<wire x1="50.8" y1="9.28" x2="50.8" y2="6.74" width="0.8128" layer="1"/>
 <via x="21" y="80.5" extent="1-16" drill="0.8" diameter="1.15"/>
 <via x="6" y="85" extent="1-16" drill="0.8" diameter="1.15"/>
@@
 <via x="80" y="40" extent="1-16" drill="0.35"/>
 <via x="86" y="37" extent="1-16" drill="0.35"/>
+<via x="32.147" y="45.323" extent="1-16" drill="0.35"/>
+<via x="37.211" y="40.894" extent="1-16" drill="0.35"/>
 </signal>
 <signal name="NRST">
@@
 <contactref element="U$4" pad="B7"/>
 <contactref element="U$4" pad="B8"/>
-<wire x1="53.38" y1="9.28" x2="53.38" y2="6.74" width="0.8128" layer="1"/>
-<wire x1="53.38" y1="9.28" x2="55.92" y2="9.28" width="0.8128" layer="1"/>
-<wire x1="55.92" y1="9.28" x2="55.92" y2="6.74" width="0.8128" layer="1"/>
-<wire x1="53.38" y1="6.74" x2="55.92" y2="6.74" width="0.8128" layer="1"/>
+<wire x1="53.34" y1="9.28" x2="53.34" y2="6.74" width="0.8128" layer="1"/>
+<wire x1="53.34" y1="9.28" x2="55.88" y2="9.28" width="0.8128" layer="1"/>
+<wire x1="55.88" y1="9.28" x2="55.88" y2="6.74" width="0.8128" layer="1"/>
+<wire x1="53.34" y1="6.74" x2="55.88" y2="6.74" width="0.8128" layer="1"/>
 <polygon width="0.508" layer="16" thermals="no">
 <vertex x="58.42" y="5.461"/>
@@
 <contactref element="U$5" pad="PA6"/>
 <wire x1="30.52" y1="58.24" x2="30.52" y2="55.84" width="0.254" layer="1"/>
-<wire x1="30.52" y1="55.84" x2="38.1" y2="48.26" width="0.254" layer="1"/>
-<wire x1="38.1" y1="48.26" x2="38.1" y2="30.48" width="0.254" layer="1"/>
-<wire x1="41.59" y1="26.99" x2="41.59" y2="25.94" width="0.254" layer="1"/>
-<wire x1="38.1" y1="30.48" x2="41.59" y2="26.99" width="0.254" layer="1"/>
+<wire x1="30.52" y1="55.84" x2="34.1" y2="52.26" width="0.254" layer="1"/>
+<wire x1="34.1" y1="52.26" x2="34.1" y2="31.48" width="0.254" layer="1"/>
+<wire x1="34.1" y1="31.48" x2="39.64" y2="25.94" width="0.254" layer="1"/>
+<wire x1="39.64" y1="25.94" x2="41.59" y2="25.94" width="0.254" layer="1"/>
 </signal>
 <signal name="TIM3_CH2">
@@
 <contactref element="U$4" pad="B11"/>
 <contactref element="U$4" pad="B12"/>
-<wire x1="43.22" y1="6.74" x2="44.45" y2="6.74" width="0.8128" layer="1"/>
-<wire x1="44.95" y1="6.74" x2="45.76" y2="6.74" width="0.8128" layer="1"/>
+<wire x1="43.18" y1="6.74" x2="44.45" y2="6.74" width="0.8128" layer="1"/>
+<wire x1="44.95" y1="6.74" x2="45.72" y2="6.74" width="0.8128" layer="1"/>
 <contactref element="U$6" pad="R3-9"/>
 <contactref element="U$6" pad="R3-1"/>
@@
 <wire x1="1.3462" y1="38.0238" x2="2.667" y2="36.703" width="0.5" layer="16"/>
 <via x="4.064" y="36.703" extent="1-16" drill="0.35"/>
-<wire x1="4.115" y1="36.652" x2="17.9956125" y2="36.652" width="0.5" layer="1"/>
 <wire x1="2.667" y1="36.703" x2="4.064" y2="36.703" width="0.5" layer="16"/>
 <wire x1="4.064" y1="36.703" x2="4.115" y2="36.652" width="0.5" layer="1"/>
 <contactref element="U$4" pad="B3"/>
 <contactref element="U$4" pad="B4"/>
-<wire x1="43.22" y1="9.28" x2="43.22" y2="6.74" width="0.8128" layer="1"/>
-<wire x1="43.22" y1="9.28" x2="45.76" y2="9.28" width="0.8128" layer="1"/>
-<wire x1="45.76" y1="9.28" x2="45.76" y2="6.74" width="0.8128" layer="1"/>
-<wire x1="45.3676125" y1="9.28" x2="45.76" y2="9.28" width="0.5" layer="1"/>
-<wire x1="17.9956125" y1="36.652" x2="45.3676125" y2="9.28" width="0.5" layer="1"/>
+<wire x1="43.18" y1="9.28" x2="43.18" y2="6.74" width="0.8128" layer="1"/>
+<wire x1="43.18" y1="9.28" x2="45.72" y2="9.28" width="0.8128" layer="1"/>
+<wire x1="45.72" y1="9.28" x2="45.72" y2="6.74" width="0.8128" layer="1"/>
+<wire x1="45.3676125" y1="9.28" x2="45.72" y2="9.28" width="0.5" layer="1"/>
+<wire x1="43.18" y1="9.28" x2="43.18" y2="10.472" width="0.508" layer="1"/>
+<wire x1="43.18" y1="10.472" x2="17" y2="36.652" width="0.508" layer="1"/>
+<wire x1="17" y1="36.652" x2="4.115" y2="36.652" width="0.508" layer="1"/>
+<wire x1="4.115" y1="36.652" x2="4.064" y2="36.703" width="0.508" layer="1"/>
 </signal>
 <signal name="+5VGND">
 <contactref element="U$4" pad="B9"/>
 <contactref element="U$4" pad="B10"/>
-<wire x1="38.14" y1="6.74" x2="39.37" y2="6.74" width="0.8128" layer="1"/>
-<wire x1="39.37" y1="6.74" x2="40.68" y2="6.74" width="0.8128" layer="1"/>
+<wire x1="38.1" y1="6.74" x2="39.37" y2="6.74" width="0.8128" layer="1"/>
+<wire x1="39.37" y1="6.74" x2="40.64" y2="6.74" width="0.8128" layer="1"/>
 <wire x1="15.755" y1="35.815" x2="39.285" y2="12.285" width="0.6096" layer="1"/>
 <wire x1="2.54" y1="35.815" x2="2.54" y2="35.8439375" width="0.508" layer="1"/>
@@
 <contactref element="U$4" pad="B1"/>
 <contactref element="U$4" pad="B2"/>
-<wire x1="38.14" y1="9.28" x2="38.14" y2="6.74" width="0.8128" layer="1"/>
-<wire x1="38.14" y1="9.28" x2="40.68" y2="9.28" width="0.8128" layer="1"/>
-<wire x1="40.68" y1="9.28" x2="40.68" y2="6.74" width="0.8128" layer="1"/>
-<wire x1="40.68" y1="10.89" x2="40.68" y2="9.28" width="0.5" layer="1"/>
+<wire x1="38.1" y1="9.28" x2="38.1" y2="6.74" width="0.8128" layer="1"/>
+<wire x1="38.1" y1="9.28" x2="40.64" y2="9.28" width="0.8128" layer="1"/>
+<wire x1="40.64" y1="9.28" x2="40.64" y2="6.74" width="0.8128" layer="1"/>
+<wire x1="40.68" y1="10.89" x2="40.64" y2="9.28" width="0.5" layer="1"/>
 <wire x1="39.285" y1="12.285" x2="39.285" y2="12.285" width="0.6096" layer="1"/>
 <wire x1="39.285" y1="12.285" x2="40.68" y2="10.89" width="0.508" layer="1"/>
@@
 <wire x1="12" y1="60.5" x2="7" y2="55.5" width="0.2032" layer="1"/>
 <wire x1="7" y1="55.5" x2="7" y2="39" width="0.2032" layer="1"/>
-<wire x1="8.5" y1="37.5" x2="18.5" y2="37.5" width="0.2032" layer="1"/>
+<wire x1="8.5" y1="37.5" x2="17.5" y2="37.5" width="0.2032" layer="1"/>
 <wire x1="7" y1="39" x2="8.5" y2="37.5" width="0.2032" layer="1"/>
-<wire x1="18.5" y1="37.5" x2="36.5" y2="19.5" width="0.2032" layer="1"/>
-<via x="36.5" y="19.5" extent="1-16" drill="0.35"/>
+<wire x1="17.5" y1="37.5" x2="36.5" y2="18.5" width="0.2032" layer="1"/>
+<via x="36.5" y="18.5" extent="1-16" drill="0.35"/>
 <wire x1="36.5" y1="17" x2="36.5" y2="4" width="0.2032" layer="16"/>
 <wire x1="36.5" y1="4" x2="38" y2="2.5" width="0.2032" layer="16"/>
 <wire x1="38" y1="2.5" x2="54.22" y2="2.5" width="0.2032" layer="16"/>
-<wire x1="54.22" y1="2.5" x2="55.92" y2="4.2" width="0.2032" layer="16"/>
-<wire x1="36.5" y1="19.5" x2="36.5" y2="17" width="0.2032" layer="16"/>
+<wire x1="54.22" y1="2.5" x2="55.88" y2="4.2" width="0.2032" layer="16"/>
+<wire x1="36.5" y1="18.5" x2="36.5" y2="17" width="0.2032" layer="16"/>
 <wire x1="8.73" y1="64.77" x2="9.21" y2="64.77" width="0.254" layer="1"/>
 <wire x1="9.93" y1="72.39" x2="9.93" y2="69.43" width="0.254" layer="1"/>
@@
 <wire x1="5.684" y1="55.184" x2="11" y2="60.5" width="0.2032" layer="1"/>
 <wire x1="11" y1="63" x2="11" y2="60.5" width="0.2032" layer="1"/>
-<wire x1="53.38" y1="4.2" x2="51.68" y2="2.5" width="0.2032" layer="1"/>
+<wire x1="53.34" y1="4.2" x2="51.68" y2="2.5" width="0.2032" layer="1"/>
 <wire x1="51.68" y1="2.5" x2="37.5" y2="2.5" width="0.2032" layer="1"/>
 <wire x1="37.5" y1="2.5" x2="36" y2="4" width="0.2032" layer="1"/>
